File: hardware/rev3/FTDI.sch (KiCad schematic (older format))
At the start: 20 parts, among them U2 93LCxxB, U3 FT2232H, Y1 12MHz

Commit message: Add AD9102 to the schematic.
Parts:
- R6: value 1k -> 4.7k
Connections:
- net ADBUS0 renamed SPI_CLK
- net ADBUS1 renamed SPI_DO
- net ADBUS2 renamed SPI_DI
- net ADBUS3 renamed SPI_CS
- net ADBUS4 renamed RESET
- net ADBUS5 renamed TRIGGER
Changed lines of the file:
@@
 LIBS:valves
 LIBS:ftdi
+LIBS:analog_devices
+LIBS:AD9102
+LIBS:LMK61XX
 LIBS:rev3-cache
 EELAYER 25 0
@@
 $Descr A4 11693 8268
 encoding utf-8
-Sheet 3 4
+Sheet 3 5
 Title ""
 Date ""
@@
 P 3100 3750
 F 0 "R6" H 3130 3770 50  0000 L CNN
-F 1 "1k" H 3130 3710 50  0000 L CNN
+F 1 "4.7k" H 3130 3710 50  0000 L CNN
 F 2 "Resistors_SMD:R_0805" H 3100 3750 50  0001 C CNN
 F 3 "" H 3100 3750 50  0001 C CNN
@@
 Connection ~ 5200 6550
 Wire Bus Line
-	6650 2450 6650 3150
+	7600 2450 7600 3150
 Wire Bus Line
 	6650 3350 6650 4050
@@
 	6550 3250 6200 3250
 Entry Wire Line
-	6550 3050 6650 3150
-Entry Wire Line
-	6550 2950 6650 3050
-Entry Wire Line
-	6550 2850 6650 2950
-Entry Wire Line
-	6550 2750 6650 2850
-Entry Wire Line
-	6550 2650 6650 2750
-Entry Wire Line
-	6550 2550 6650 2650
-Entry Wire Line
-	6550 2450 6650 2550
-Entry Wire Line
-	6550 2350 6650 2450
-Wire Wire Line
-	6200 2350 6550 2350
-Wire Wire Line
-	6550 2450 6200 2450
-Wire Wire Line
-	6200 2550 6550 2550
-Wire Wire Line
-	6550 2650 6200 2650
-Wire Wire Line
-	6200 2750 6550 2750
-Wire Wire Line
-	6550 2850 6200 2850
-Wire Wire Line
-	6200 2950 6550 2950
-Wire Wire Line
-	6550 3050 6200 3050
+	7500 3050 7600 3150
+Entry Wire Line
+	7500 2950 7600 3050
+Entry Wire Line
+	7500 2850 7600 2950
+Entry Wire Line
+	7500 2750 7600 2850
+Entry Wire Line
+	7500 2650 7600 2750
+Entry Wire Line
+	7500 2550 7600 2650
+Entry Wire Line
+	7500 2450 7600 2550
+Entry Wire Line
+	7500 2350 7600 2450
+Wire Wire Line
+	6200 2350 7500 2350
+Wire Wire Line
+	6200 2450 7500 2450
+Wire Wire Line
+	6200 2550 7500 2550
+Wire Wire Line
+	6200 2650 7500 2650
+Wire Wire Line
+	6200 2750 7500 2750
+Wire Wire Line
+	6200 2850 7500 2850
+Wire Wire Line
+	6200 2950 7500 2950
+Wire Wire Line
+	6200 3050 7500 3050
 Wire Bus Line
 	6650 4250 6650 4950
@@
 Text Label 6200 3050 0    60   ~ 0
 ADBUS7
-Text HLabel 6650 2450 2    60   Input ~ 0
+Text HLabel 7600 2450 2    60   Input ~ 0
 ADBUS[7..0]
 Text HLabel 6650 3350 2    60   Input ~ 0
@@
 Text Label 6200 5750 0    60   ~ 0
 BCBUS7
+Text GLabel 6650 2200 1    60   Input ~ 0
+SPI_CLK
+Text GLabel 6800 2200 1    60   Input ~ 0
+SPI_DO
+Text GLabel 6950 2200 1    60   Input ~ 0
+SPI_DI
+Text GLabel 7100 2200 1    60   Input ~ 0
+SPI_CS
+Wire Wire Line
+	6650 2200 6650 2350
+Connection ~ 6650 2350
+Wire Wire Line
+	6800 2200 6800 2450
+Connection ~ 6800 2450
+Wire Wire Line
+	6950 2200 6950 2550
+Connection ~ 6950 2550
+Wire Wire Line
+	7100 2200 7100 2650
+Connection ~ 7100 2650
+Text GLabel 7250 2200 1    60   Input ~ 0
+RESET
+Wire Wire Line
+	7250 2200 7250 2750
+Connection ~ 7250 2750
+Text GLabel 7400 2200 1    60   Input ~ 0
+TRIGGER
+Wire Wire Line
+	7400 2200 7400 2850
+Connection ~ 7400 2850
 $EndSCHEMATC

Commit message: Finish up output amp schematic.
Parts:
- renumbered C12 to C10, C13 to C11, C14 to C12, C15 to C13, C16 to C14, C17 to C15, C7 to C16, C8 to C17, C9 to C7, C10 to C8, C11 to C9, R5 to R3, R2 to R4, R3 to R5, R4 to R6, R6 to R7, R7 to R8
Connections:
- net ADBUS6 renamed AMP0_EN
- net ADBUS7 renamed AMP1_EN

Commit message: Add missing footprints.
Parts:
- C10, C11, C12, C13, C14, C15, C16, C17, C7, C8, C9: footprint Capacitors_SMD:C_0805 -> Capacitors_SMD:C_0603_HandSoldering
- R3, R4, R5, R6, R7, R8: footprint Resistors_SMD:R_0805 -> Resistors_SMD:R_0603_HandSoldering
Changed lines of the file:
@@
 F 0 "R4" H 1230 1320 50  0000 L CNN
 F 1 "10k" H 1230 1260 50  0000 L CNN
-F 2 "Resistors_SMD:R_0805" H 1200 1300 50  0001 C CNN
+F 2 "Resistors_SMD:R_0603_HandSoldering" H 1200 1300 50  0001 C CNN
 F 3 "" H 1200 1300 50  0001 C CNN
 F 4 "P10KADCT-ND" H 1200 1300 60  0001 C CNN "DigiKey "
@@
 F 0 "R5" H 1430 1320 50  0000 L CNN
 F 1 "10k" H 1430 1260 50  0000 L CNN
-F 2 "Resistors_SMD:R_0805" H 1400 1300 50  0001 C CNN
+F 2 "Resistors_SMD:R_0603_HandSoldering" H 1400 1300 50  0001 C CNN
 F 3 "" H 1400 1300 50  0001 C CNN
 F 4 "P10KADCT-ND" H 1400 1300 60  0001 C CNN "DigiKey "
@@
 F 0 "R3" H 2530 1270 50  0000 L CNN
 F 1 "10k" H 2530 1210 50  0000 L CNN
-F 2 "Resistors_SMD:R_0805" H 2500 1250 50  0001 C CNN
+F 2 "Resistors_SMD:R_0603_HandSoldering" H 2500 1250 50  0001 C CNN
 F 3 "" H 2500 1250 50  0001 C CNN
 F 4 "P10KADCT-ND" H 2500 1250 60  0001 C CNN "DigiKey "
@@
 F 0 "R6" H 2380 1720 50  0000 L CNN
 F 1 "2.2k" H 2380 1660 50  0000 L CNN
-F 2 "Resistors_SMD:R_0805" H 2350 1700 50  0001 C CNN
+F 2 "Resistors_SMD:R_0603_HandSoldering" H 2350 1700 50  0001 C CNN
 F 3 "" H 2350 1700 50  0001 C CNN
 F 4 "P2.2KADCT-ND" H 2350 1700 60  0001 C CNN "DigiKey "
@@
 F 0 "C8" H 1960 2820 50  0000 L CNN
 F 1 "100n" H 1960 2670 50  0000 L CNN
-F 2 "Capacitors_SMD:C_0805" H 1950 2750 50  0001 C CNN
+F 2 "Capacitors_SMD:C_0603_HandSoldering" H 1950 2750 50  0001 C CNN
 F 3 "" H 1950 2750 50  0001 C CNN
 F 4 "478-1395-1-ND" H 1950 2750 60  0001 C CNN "DigiKey "
@@
 F 0 "C9" H 2210 2820 50  0000 L CNN
 F 1 "100n" H 2210 2670 50  0000 L CNN
-F 2 "Capacitors_SMD:C_0805" H 2200 2750 50  0001 C CNN
+F 2 "Capacitors_SMD:C_0603_HandSoldering" H 2200 2750 50  0001 C CNN
 F 3 "" H 2200 2750 50  0001 C CNN
 F 4 "478-1395-1-ND" H 2200 2750 60  0001 C CNN "DigiKey "
@@
 F 0 "C10" H 2460 2820 50  0000 L CNN
 F 1 "100n" H 2460 2670 50  0000 L CNN
-F 2 "Capacitors_SMD:C_0805" H 2450 2750 50  0001 C CNN
+F 2 "Capacitors_SMD:C_0603_HandSoldering" H 2450 2750 50  0001 C CNN
 F 3 "" H 2450 2750 50  0001 C CNN
 F 4 "478-1395-1-ND" H 2450 2750 60  0001 C CNN "DigiKey "
@@
 F 0 "C11" H 2710 2820 50  0000 L CNN
 F 1 "100n" H 2710 2670 50  0000 L CNN
-F 2 "Capacitors_SMD:C_0805" H 2700 2750 50  0001 C CNN
+F 2 "Capacitors_SMD:C_0603_HandSoldering" H 2700 2750 50  0001 C CNN
 F 3 "" H 2700 2750 50  0001 C CNN
 F 4 "478-1395-1-ND" H 2700 2750 60  0001 C CNN "DigiKey "
@@
 F 0 "C12" H 2960 2820 50  0000 L CNN
 F 1 "100n" H 2960 2670 50  0000 L CNN
-F 2 "Capacitors_SMD:C_0805" H 2950 2750 50  0001 C CNN
+F 2 "Capacitors_SMD:C_0603_HandSoldering" H 2950 2750 50  0001 C CNN
 F 3 "" H 2950 2750 50  0001 C CNN
 F 4 "478-1395-1-ND" H 2950 2750 60  0001 C CNN "DigiKey "
@@
 F 0 "C13" H 3210 2820 50  0000 L CNN
 F 1 "100n" H 3210 2670 50  0000 L CNN
-F 2 "Capacitors_SMD:C_0805" H 3200 2750 50  0001 C CNN
+F 2 "Capacitors_SMD:C_0603_HandSoldering" H 3200 2750 50  0001 C CNN
 F 3 "" H 3200 2750 50  0001 C CNN
 F 4 "478-1395-1-ND" H 3200 2750 60  0001 C CNN "DigiKey "
@@
 F 0 "C14" H 3460 2820 50  0000 L CNN
 F 1 "100n" H 3460 2670 50  0000 L CNN
-F 2 "Capacitors_SMD:C_0805" H 3450 2750 50  0001 C CNN
+F 2 "Capacitors_SMD:C_0603_HandSoldering" H 3450 2750 50  0001 C CNN
 F 3 "" H 3450 2750 50  0001 C CNN
 F 4 "478-1395-1-ND" H 3450 2750 60  0001 C CNN "DigiKey "
@@
 F 0 "C7" H 1710 2820 50  0000 L CNN
 F 1 "3.3u" H 1710 2670 50  0000 L CNN
-F 2 "Capacitors_SMD:C_0805" H 1700 2750 50  0001 C CNN
+F 2 "Capacitors_SMD:C_0603_HandSoldering" H 1700 2750 50  0001 C CNN
 F 3 "" H 1700 2750 50  0001 C CNN
 F 4 "478-1414-1-ND" H 1700 2750 60  0001 C CNN "DigiKey "
@@
 F 0 "C15" H 3710 2820 50  0000 L CNN
 F 1 "100n" H 3710 2670 50  0000 L CNN
-F 2 "Capacitors_SMD:C_0805" H 3700 2750 50  0001 C CNN
+F 2 "Capacitors_SMD:C_0603_HandSoldering" H 3700 2750 50  0001 C CNN
 F 3 "" H 3700 2750 50  0001 C CNN
 F 4 "478-1395-1-ND" H 3700 2750 60  0001 C CNN "DigiKey "
@@
 F 0 "R7" H 3130 3770 50  0000 L CNN
 F 1 "4.7k" H 3130 3710 50  0000 L CNN
-F 2 "Resistors_SMD:R_0805" H 3100 3750 50  0001 C CNN
+F 2 "Resistors_SMD:R_0603_HandSoldering" H 3100 3750 50  0001 C CNN
 F 3 "" H 3100 3750 50  0001 C CNN
 F 4 "P1.0KADCT-ND" H 3100 3750 60  0001 C CNN "DigiKey "
@@
 F 0 "R8" H 3680 4020 50  0000 L CNN
 F 1 "12k" H 3680 3960 50  0000 L CNN
-F 2 "Resistors_SMD:R_0805" H 3650 4000 50  0001 C CNN
+F 2 "Resistors_SMD:R_0603_HandSoldering" H 3650 4000 50  0001 C CNN
 F 3 "" H 3650 4000 50  0001 C CNN
 F 4 "P12KADCT-ND" H 3650 4000 60  0001 C CNN "DigiKey "
@@
 F 0 "C16" H 1160 6520 50  0000 L CNN
 F 1 "27p" H 1160 6370 50  0000 L CNN
-F 2 "Capacitors_SMD:C_0805" H 1150 6450 50  0001 C CNN
+F 2 "Capacitors_SMD:C_0603_HandSoldering" H 1150 6450 50  0001 C CNN
 F 3 "" H 1150 6450 50  0001 C CNN
 F 4 "478-10518-1-ND" H 1150 6450 60  0001 C CNN "DigiKey "
@@
 F 0 "C17" H 1660 6520 50  0000 L CNN
 F 1 "27p" H 1660 6370 50  0000 L CNN
-F 2 "Capacitors_SMD:C_0805" H 1650 6450 50  0001 C CNN
+F 2 "Capacitors_SMD:C_0603_HandSoldering" H 1650 6450 50  0001 C CNN
 F 3 "" H 1650 6450 50  0001 C CNN
 F 4 "478-10518-1-ND" H 1650 6450 60  0001 C CNN "DigiKey "
