File: hardware/rev3/rev3.kicad_pcb (KiCad board)
At the start: 2 copper layers, 37 parts, among them J1 USB_B, J2 CONN_02X09, J3 CONN_02X09, U1 LD1117S33TR, U2 93LCxxB, U3 FT2232H, Y1 12MHz

Commit message: Make some progress on layout.
Parts:
- added C18: DNP, Capacitors_SMD:C_0603_HandSoldering, F.Cu at (35.1, 42.7)
- added C19: DNP, Capacitors_SMD:C_0603_HandSoldering, F.Cu at (46.7, 45.7)
- added C20: DNP, Capacitors_SMD:C_0603_HandSoldering, F.Cu at (46.8, 41.1)
- added C21: DNP, Capacitors_SMD:C_0603_HandSoldering, F.Cu at (43.2, 43.2)
- added C22: 10u, Capacitors_SMD:C_0603_HandSoldering, F.Cu at (94.6, 147.5)
- added C23: 100n, Capacitors_SMD:C_0603_HandSoldering, F.Cu at (98.7, 142.7)
- added C24: 100n, Capacitors_SMD:C_0603_HandSoldering, F.Cu at (105.1, 137.6)
- added C25: 100n, Capacitors_SMD:C_0603_HandSoldering, F.Cu at (101.0, 137.6)
- added C26: 0.8p, Capacitors_SMD:C_0603_HandSoldering, F.Cu at (115.9, 122.7)
- added C27: 2.8p, Capacitors_SMD:C_0603_HandSoldering, F.Cu at (94.6, 142.7)
- added C28: 100n, Capacitors_SMD:C_0603_HandSoldering, F.Cu at (105.4, 132.3)
- added C29: 10u, Capacitors_SMD:C_0603_HandSoldering, F.Cu at (109.4, 127.5)
- added C30: 100n, Capacitors_SMD:C_0603_HandSoldering, F.Cu at (90.5, 147.7)
- added C31: 2.8p, Capacitors_SMD:C_0603_HandSoldering, F.Cu at (111.8, 122.7)
- added C32: 0.8p, Capacitors_SMD:C_0603_HandSoldering, F.Cu at (105.4, 127.5)
- added C33: 100n, Capacitors_SMD:C_0603_HandSoldering, F.Cu at (101.2, 132.8)
- added C34: 10u, Capacitors_SMD:C_0603_HandSoldering, F.Cu at (103.7, 122.7)
- added C35: 100n, Capacitors_SMD:C_0603_HandSoldering, F.Cu at (109.6, 132.3)
- added C36: 100n, Capacitors_SMD:C_0603_HandSoldering, F.Cu at (96.8, 137.9)
- added C37: 100n, Capacitors_SMD:C_0603_HandSoldering, F.Cu at (86.4, 148.5)
- added C38: 100n, Capacitors_SMD:C_0603_HandSoldering, F.Cu at (90.5, 142.9)
- added C39: 100n, Capacitors_SMD:C_0603_HandSoldering, F.Cu at (86.4, 143.7)
- added C40: 100n, Capacitors_SMD:C_0603_HandSoldering, F.Cu at (92.7, 137.9)
- added C41: 100n, Capacitors_SMD:C_0603_HandSoldering, F.Cu at (97.0, 132.8)
- added C42: 10u, Capacitors_SMD:C_0603_HandSoldering, F.Cu at (101.3, 127.8)
- added C43: 1u, Capacitors_SMD:C_0603_HandSoldering, F.Cu at (107.8, 122.7)
- added C44: 100n, Capacitors_SMD:C_0603_HandSoldering, F.Cu at (82.0, 148.8)
- added J4: SMA, Connectors_Molex:Molex_SMA_Jack_Edge_Mount, F.Cu at (149.9, 104.7)
- added J5: CONN_02X09, Pin_Headers:Pin_Header_Straight_2x09_Pitch2.54mm, F.Cu at (175.3, 74.2)
- added J6: SMA, Connectors_Molex:Molex_SMA_Jack_Edge_Mount, F.Cu at (162.6, 104.7)
- added J7: SMA, Connectors_Molex:Molex_SMA_Jack_Edge_Mount, F.Cu at (137.2, 104.7)
- added JP1: USB_PWR, Pin_Headers:Pin_Header_Straight_1x02_Pitch2.54mm, F.Cu at (153.9, 40.1)
- added L3: 800m, Inductors_SMD:L_0603_HandSoldering, F.Cu at (75.2, 130.1)
- added L4: 800m, Inductors_SMD:L_0603_HandSoldering, F.Cu at (81.9, 123.4)
- added R10: DNP, Resistors_SMD:R_0603_HandSoldering, F.Cu at (79.7, 134.7)
- added R11: 8k, Resistors_SMD:R_0603_HandSoldering, F.Cu at (73.2, 145.6)
- added R12: 500, Resistors_SMD:R_0603_HandSoldering, F.Cu at (84.0, 138.9)
- added R13: 4.7k, Resistors_SMD:R_0603_HandSoldering, F.Cu at (99.5, 122.9)
- added R14: 1.5k, Resistors_SMD:R_0603_HandSoldering, F.Cu at (77.8, 144.8)
- added R15: 100, Resistors_SMD:R_0603_HandSoldering, F.Cu at (82.1, 143.9)
- added R16: 4.7k, Resistors_SMD:R_0603_HandSoldering, F.Cu at (95.1, 122.9)
- added R17: 4.7k, Resistors_SMD:R_0603_HandSoldering, F.Cu at (88.4, 133.0)
- added R18: 1k, Resistors_SMD:R_0603_HandSoldering, F.Cu at (77.8, 139.8)
- added R19: 100, Resistors_SMD:R_0603_HandSoldering, F.Cu at (88.4, 128.0)
- added R20: 100, Resistors_SMD:R_0603_HandSoldering, F.Cu at (84.0, 133.8)
- added R21: 1k, Resistors_SMD:R_0603_HandSoldering, F.Cu at (90.8, 122.9)
- added R22: 100, Resistors_SMD:R_0603_HandSoldering, F.Cu at (86.4, 122.9)
- added R23: 1.5k, Resistors_SMD:R_0603_HandSoldering, F.Cu at (73.4, 140.6)
- added R24: 100, Resistors_SMD:R_0603_HandSoldering, F.Cu at (73.4, 135.5)
- added R25: 4.7k, Resistors_SMD:R_0603_HandSoldering, F.Cu at (79.7, 129.7)
- added R26: 10k, Resistors_SMD:R_0603_HandSoldering, F.Cu at (92.8, 133.0)
- added R27: 500, Resistors_SMD:R_0603_HandSoldering, F.Cu at (88.4, 138.1)
- added R28: 10k, Resistors_SMD:R_0603_HandSoldering, F.Cu at (97.1, 128.0)
- added R29: 4.7k, Resistors_SMD:R_0603_HandSoldering, F.Cu at (92.8, 128.0)
- added R8: 12k, Resistors_SMD:R_0603_HandSoldering, F.Cu at (95.2, 12.6)
- added R9: DNP, Resistors_SMD:R_0603_HandSoldering, F.Cu at (84.0, 128.8)
- added REF**: MountingHole_3.5mm_Pad_Via, Mounting_Holes:MountingHole_3.5mm_Pad_Via, F.Cu at (127.0, 38.1)
- added REF**: MountingHole_3.5mm_Pad_Via, Mounting_Holes:MountingHole_3.5mm_Pad_Via, F.Cu at (172.7, 38.1)
- added REF**: MountingHole_3.5mm_Pad_Via, Mounting_Holes:MountingHole_3.5mm_Pad_Via, F.Cu at (127.0, 104.1)
- added REF**: MountingHole_3.5mm_Pad_Via, Mounting_Holes:MountingHole_3.5mm_Pad_Via, F.Cu at (172.7, 104.1)
- added TP4: TRIGGER, Measurement_Points:Test_Point_Keystone_5005-5009_Compact, F.Cu at (99.6, 81.3)
- added TP5: VOUT+, Measurement_Points:Test_Point_Keystone_5005-5009_Compact, F.Cu at (149.9, 99.6)
- added TP6: VOUT-, Measurement_Points:Test_Point_Keystone_5005-5009_Compact, F.Cu at (162.6, 99.6)
- added TP7: VOUT, Measurement_Points:Test_Point_Keystone_5005-5009_Compact, F.Cu at (137.2, 99.6)
- added U4: LTC6409, footprints:LTC6409-UDB, F.Cu at (67.7, 143.6)
- added U5: LTC6269, footprints:LTC6269-10DFN, F.Cu at (76.2, 123.8)
- added U6: AD9102, footprints:AD9102-10LFCSP, F.Cu at (68.2, 135.5)
- added X1: DSC1123, footprints:7050XO, F.Cu at (67.6, 124.1)
- C1: value 4.7u -> 100n; footprint Capacitors_SMD:C_0805 -> Capacitors_SMD:C_0603_HandSoldering
- C10, C11, C12, C13, C14, C15, C3, C4: footprint Capacitors_SMD:C_0805 -> Capacitors_SMD:C_0603_HandSoldering
- C16, C17: value 100n -> 27p; footprint Capacitors_SMD:C_0805 -> Capacitors_SMD:C_0603_HandSoldering
- C2: value 100n -> 100u; footprint Capacitors_SMD:C_0805 -> Capacitors_SMD:C_0603_HandSoldering
- C5: value 100n -> 4.7u; footprint Capacitors_SMD:C_0805 -> Capacitors_SMD:C_0603_HandSoldering
- C6: value 100u -> 100n; footprint Capacitors_SMD:C_0805 -> Capacitors_SMD:C_0603_HandSoldering
- C7: value 27p -> 3.3u; footprint Capacitors_SMD:C_0805 -> Capacitors_SMD:C_0603_HandSoldering
- C8: value 27p -> 100n; footprint Capacitors_SMD:C_0805 -> Capacitors_SMD:C_0603_HandSoldering
- C9: value 3.3u -> 100n; footprint Capacitors_SMD:C_0805 -> Capacitors_SMD:C_0603_HandSoldering
- J2: value CONN_02X09 -> SMA; footprint Pin_Headers:Pin_Header_Straight_2x09_Pitch2.54mm -> Connectors:SMA_THT_Jack_Straight
- L1, L2: footprint Inductors_SMD:L_0805 -> Inductors_SMD:L_0603_HandSoldering
- R1: value 470 -> DNP; footprint Resistors_SMD:R_0805 -> Resistors_SMD:R_0603_HandSoldering
- R2: value 10k -> 470; footprint Resistors_SMD:R_0805 -> Resistors_SMD:R_0603_HandSoldering
- R3, R5: footprint Resistors_SMD:R_0805 -> Resistors_SMD:R_0603_HandSoldering
- R4: value 2.2k -> 10k; footprint Resistors_SMD:R_0805 -> Resistors_SMD:R_0603_HandSoldering
- R6: value 1k -> 2.2k; footprint Resistors_SMD:R_0805 -> Resistors_SMD:R_0603_HandSoldering
- R7: value 12k -> 4.7k; footprint Resistors_SMD:R_0805 -> Resistors_SMD:R_0603_HandSoldering
- TP2: value GND -> +3.3V
- TP3: value +3.3V -> GND
- moved D1 160.1 mm to (80.9, 51.6)
- moved C14 158.1 mm to (99.4, 12.4)
- moved R4 156.6 mm to (90.8, 12.6)
- moved C11 153.7 mm to (94.9, 17.4)
- moved R3 153.4 mm to (64.2, 31.3)
- moved C15 153.4 mm to (90.7, 17.4)
- moved C2 153.3 mm to (83.5, 56.9)
- moved C13 152.7 mm to (77.2, 31.1)
- moved C16 152.2 mm to (97.7, 22.2)
- moved R5 149.4 mm to (68.6, 31.3)
- moved C10 149.2 mm to (99.0, 17.4)
- moved Y1 148.8 mm to (84.0, 23.0)
- moved C8 148.2 mm to (93.6, 22.2)
- moved C9 148.0 mm to (89.4, 22.2)
- moved C17 146.5 mm to (93.4, 27.0)
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Connections:
- C1 pad 1: FTVPHY -> Net-(C1-Pad1)
- C1 pad 2: GNDD -> GNDA
- C10 pad 2: GNDD -> GNDA
- C11 pad 2: GNDD -> GNDA
- C12 pad 2: GNDD -> GNDA
- C13 pad 2: GNDD -> GNDA
- C14 pad 2: GNDD -> GNDA
- C15 pad 1: /FTDI/VREGOUT -> +3V3
- C15 pad 2: GNDD -> GNDA
- C16 pad 1: /FTDI/VREGOUT -> FTOSC+
- C16 pad 2: GNDD -> GNDA
- C17 pad 1: +3V3 -> FTOSC-
- C17 pad 2: GNDD -> GNDA
- C2 pad 1: FTVPHY -> +3V3
- C2 pad 2: GNDD -> GNDA
- C3 pad 1: FTVPLL -> FTVPHY
- C3 pad 2: GNDD -> GNDA
- C4 pad 1: FTVPLL -> FTVPHY
- C4 pad 2: GNDD -> GNDA
- C5 pad 1: Net-(C5-Pad1) -> FTVPLL
- C5 pad 2: GNDD -> GNDA
- C6 pad 1: +3V3 -> FTVPLL
- C6 pad 2: GNDD -> GNDA
- C7 pad 1: FTOSC+ -> /FTDI/VREGOUT
- C7 pad 2: GNDD -> GNDA
- C8 pad 1: FTOSC- -> /FTDI/VREGOUT
- C8 pad 2: GNDD -> GNDA
- C9 pad 2: GNDD -> GNDA
- D1 pad 1: GNDD -> GNDA
- J1 pad 1: Net-(C5-Pad1) -> Net-(J1-Pad1)
- J1 pad 4: GNDD -> GNDA
- J2 pad 1: +3V3 -> TRIGGER
- J2 pad 2: GNDD -> GNDA
- J3 pad 10: /Connectors/BCBUS3 -> /Connectors/ACBUS3
- J3 pad 11: /Connectors/BDBUS4 -> RESET
- J3 pad 12: /Connectors/BCBUS4 -> /Connectors/ACBUS4
- J3 pad 13: /Connectors/BDBUS5 -> TRIGGER
- J3 pad 14: /Connectors/BCBUS5 -> /Connectors/ACBUS5
- J3 pad 15: /Connectors/BDBUS6 -> AMP0_EN
- J3 pad 16: /Connectors/BCBUS6 -> /Connectors/ACBUS6
- J3 pad 17: /Connectors/BDBUS7 -> AMP1_EN
- J3 pad 18: /Connectors/BCBUS7 -> /Connectors/ACBUS7
- J3 pad 2: GNDD -> GNDA
- J3 pad 3: /Connectors/BDBUS0 -> SPI_CLK
- J3 pad 4: /Connectors/BCBUS0 -> /Connectors/ACBUS0
- J3 pad 5: /Connectors/BDBUS1 -> SPI_DO
- J3 pad 6: /Connectors/BCBUS1 -> /Connectors/ACBUS1
- J3 pad 7: /Connectors/BDBUS2 -> SPI_DI
- J3 pad 8: /Connectors/BCBUS2 -> /Connectors/ACBUS2
- J3 pad 9: /Connectors/BDBUS3 -> SPI_CS
- R1 pad 1: +3V3 -> GNDA
- R1 pad 2: Net-(D1-Pad2) -> Net-(J1-Pad5)
- R2 pad 2: FTEECLK -> Net-(D1-Pad2)
- R3 pad 2: FTEECS -> FTEEDATA
- R4 pad 1: FTEEDATA -> +3V3
- R4 pad 2: Net-(R4-Pad2) -> FTEECLK
- R5 pad 2: FTEEDATA -> FTEECS
- R6 pad 1: +3V3 -> FTEEDATA
- R6 pad 2: /FTDI/nRESET -> Net-(R6-Pad2)
- R7 pad 1: GNDD -> +3V3
- R7 pad 2: /FTDI/REF -> /FTDI/nRESET
- TP1 pad 1: Net-(C5-Pad1) -> Net-(C1-Pad1)
- TP2 pad 1: GNDD -> +3V3
- TP3 pad 1: +3V3 -> GNDA
- U1 pad 1: GNDD -> GNDA
- U1 pad 3: Net-(C5-Pad1) -> Net-(C1-Pad1)
- U2 pad 4: Net-(R4-Pad2) -> Net-(R6-Pad2)
- U2 pad 5: GNDD -> GNDA
- U2 pad 6: Net-(U2-Pad6) -> (no net)
- U2 pad 7: Net-(U2-Pad7) -> (no net)
- U3 pad 1: GNDD -> GNDA
- U3 pad 10: GNDD -> GNDA
- U3 pad 11: GNDD -> GNDA
- U3 pad 13: GNDD -> GNDA
- U3 pad 15: GNDD -> GNDA
- U3 pad 16: /Connectors/ADBUS0 -> SPI_CLK
- U3 pad 17: /Connectors/ADBUS1 -> SPI_DO
- U3 pad 18: /Connectors/ADBUS2 -> SPI_DI
- U3 pad 19: /Connectors/ADBUS3 -> SPI_CS
- U3 pad 21: /Connectors/ADBUS4 -> RESET
- U3 pad 22: /Connectors/ADBUS5 -> TRIGGER
- U3 pad 23: /Connectors/ADBUS6 -> AMP0_EN
- U3 pad 24: /Connectors/ADBUS7 -> AMP1_EN
- U3 pad 25: GNDD -> GNDA
- U3 pad 35: GNDD -> GNDA
- U3 pad 36: Net-(U3-Pad36) -> (no net)
- U3 pad 47: GNDD -> GNDA
- U3 pad 5: GNDD -> GNDA
- U3 pad 51: GNDD -> GNDA
- U3 pad 60: Net-(U3-Pad60) -> (no net)
Other:
- board outline added: 55.9 x 76.2 mm
- copper layers 2 -> 4

Commit message: Initial placement.
Parts:
- added C45: 4.7u, Capacitors_SMD:C_0603_HandSoldering, F.Cu at (189.4, 93.0)
- added C46: 1u, Capacitors_SMD:C_0603_HandSoldering, F.Cu at (189.7, 96.5)
- added C47: 100n, Capacitors_SMD:C_0603_HandSoldering, F.Cu at (156.9, 43.9)
- added R30: 50k, Resistors_SMD:R_0603_HandSoldering, F.Cu at (189.5, 91.7)
- C2: value 100u -> 10u
- J1: footprint WG:USB_Micro-B-circular -> footprints:USB_Micro-B-circular
- R26, R28: value 10k -> 100k
- X1: footprint footprints:7050XO -> footprints:3225XO
- moved C20 134.3 mm to (166.9, 101.3), turned to 180 degrees
- moved R14 130.0 mm to (192.6, 83.8), turned to 180 degrees
- moved R23 123.9 mm to (185.6, 88.1), turned to 270 degrees
- moved C19 121.0 mm to (154.2, 101.3), turned to 180 degrees
- moved U5 120.1 mm to (190.7, 87.9), turned to 180 degrees
- moved R25 118.4 mm to (188.7, 83.7), turned to 90 degrees
- moved C27 114.9 mm to (192.6, 82.5)
- moved C21 114.2 mm to (141.5, 101.3), turned to 180 degrees
- moved U4 107.2 mm to (157.8, 85.6), turned to 270 degrees
- moved C18 103.9 mm to (133.4, 75.9), turned to 180 degrees
- moved R3 101.7 mm to (162.8, 56.3), turned to 135 degrees
- moved R26 101.3 mm to (186.9, 95.6), turned to 270 degrees
- moved J2 100.7 mm to (131.1, 80.8)
- moved R18 99.1 mm to (161.6, 87.0)
- moved R28 96.8 mm to (188.3, 95.6), turned to 90 degrees
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Connections:
- R22 pad 1: GNDA -> Net-(R19-Pad2)
- REF** pad 1: (no net) -> GNDA (x4)
- U5 pad 8: Net-(C31-Pad1) -> Net-(R30-Pad1)
Routing:
- net USB_D+: track 0.00 -> 25.2 mm
- net USB_D-: track 0.00 -> 24.6 mm
- net FTOSC+: track 0.00 -> 11.2 mm
- net FTOSC-: track 0.00 -> 10.5 mm
- net GNDA: track 0.00 -> 1.53 mm, vias 0 -> 1
- added copper zone on In2.Cu, net +3V3
- added copper zone on In1.Cu, net GNDA
Other:
- net class 100ish_ohm added: clearance 0.635, trace_width 0.1778, via_dia 0.6096, via_drill 0.4064
- net class 100ohm_diff added: clearance 0.1905, trace_width 0.3429, via_dia 0.6096, via_drill 0.4064
- net class 50ohm added: clearance 0.635, trace_width 0.36195, via_dia 0.6096, via_drill 0.4064
- net class Default: clearance 0.2 -> 0.1905; trace_width 0.25 -> 0.254; via_dia 0.6 -> 0.6096; via_drill 0.4 -> 0.4064
- rule trace_clearance: 0.2 -> 0.1905
- rule trace_min: 0.2 -> 0.1524
- rule via_min_drill: 0.3 -> 0.4064
- rule via_min_size: 0.4 -> 0.6096

Commit message: First routing attempt.
Parts:
- moved C29 53.1 mm to (140.8, 98.9)
- moved C28 53.1 mm to (140.8, 100.2)
- moved C46 52.2 mm to (137.5, 95.6), turned to 180 degrees
- moved C27 51.3 mm to (144.4, 100.2), turned to 180 degrees
- moved R28 50.8 mm to (137.5, 96.8), turned to 180 degrees
- moved R14 50.6 mm to (144.4, 99.1), turned to 0 degrees
- moved R26 49.4 mm to (137.5, 94.3), turned to 0 degrees
- moved U5 48.9 mm to (142.6, 96.6), turned to 90 degrees
- moved R25 47.9 mm to (142.1, 94.4), turned to 0 degrees
- moved R30 47.4 mm to (142.0, 92.4)
- moved C31 42.0 mm to (145.4, 93.6), turned to 270 degrees
- moved C45 41.5 mm to (147.9, 93.6), turned to 270 degrees
- moved R23 39.4 mm to (146.7, 93.6), turned to 90 degrees
- moved R21 19.2 mm to (146.7, 96.4), turned to 180 degrees
- moved R18 18.3 mm to (146.6, 97.5), turned to 180 degrees
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Connections:
- net Net-(C31-Pad1) renamed /Analog/+1.65V
- REF** pad : (no net) -> GNDA (x4)
Routing:
- net GNDA: track 1.53 -> 101.9 mm, vias 1 -> 33
- net +3V3: track 0.00 -> 48.3 mm, vias 0 -> 24
- net TRIGGER: track 0.00 -> 43.5 mm, vias 0 -> 2
- net SPI_CLK: track 0.00 -> 43.0 mm, vias 0 -> 2
- net /FTDI/VREGOUT: track 0.00 -> 42.4 mm
- net AMP0_EN: track 0.00 -> 39.0 mm
- net SPI_DO: track 0.00 -> 38.0 mm, vias 0 -> 2
- net AMP1_EN: track 0.00 -> 37.1 mm
- net SPI_CS: track 0.00 -> 37.1 mm, vias 0 -> 2
- net SPI_DI: track 0.00 -> 36.7 mm, vias 0 -> 2
- net RESET: track 0.00 -> 36.6 mm, vias 0 -> 2
- net Net-(L3-Pad1): track 0.00 -> 33.9 mm, vias 0 -> 3
- net /Connectors/ACBUS7: track 0.00 -> 33.6 mm, vias 0 -> 1
- net /Connectors/ACBUS6: track 0.00 -> 31.1 mm, vias 0 -> 1
- net /Connectors/ACBUS0: track 0.00 -> 31.0 mm, vias 0 -> 1
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Other:
- rule via_min_drill: 0.4064 -> 0.3556
- rule via_min_size: 0.6096 -> 0.5588

Commit message: Update component selection based on digikey availability.
Parts:
- R11: value 8k -> 8.25k
- R12, R27: value 500 -> 510
- R2: value 470 -> 500
- R26, R28: value 100k -> 36k
- R30: value 50k -> 18k
Changed lines of the file:
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@@
       (effects (font (size 1 1) (thickness 0.15)))
     )
-    (fp_text value 470 (at 0 1.55 270) (layer F.Fab)
+    (fp_text value 500 (at 0 1.55 270) (layer F.Fab)
       (effects (font (size 1 1) (thickness 0.15)))
     )
@@
       (effects (font (size 1 1) (thickness 0.15)))
     )
-    (fp_text value 8k (at 0 1.55 90) (layer F.Fab)
+    (fp_text value 8.25k (at 0 1.55 90) (layer F.Fab)
       (effects (font (size 1 1) (thickness 0.15)))
     )
@@
       (effects (font (size 1 1) (thickness 0.15)))
     )
-    (fp_text value 500 (at 0 1.55 270) (layer F.Fab)
+    (fp_text value 510 (at 0 1.55 270) (layer F.Fab)
       (effects (font (size 1 1) (thickness 0.15)))
     )
@@
       (effects (font (size 1 1) (thickness 0.15)))
     )
-    (fp_text value 100k (at 0 1.55) (layer F.Fab)
+    (fp_text value 36k (at 0 1.55) (layer F.Fab)
       (effects (font (size 1 1) (thickness 0.15)))
     )
@@
       (effects (font (size 1 1) (thickness 0.15)))
     )
-    (fp_text value 500 (at 0 1.55 270) (layer F.Fab)
+    (fp_text value 510 (at 0 1.55 270) (layer F.Fab)
       (effects (font (size 1 1) (thickness 0.15)))
     )
@@
       (effects (font (size 1 1) (thickness 0.15)))
     )
-    (fp_text value 100k (at 0 1.55 180) (layer F.Fab)
+    (fp_text value 36k (at 0 1.55 180) (layer F.Fab)
       (effects (font (size 1 1) (thickness 0.15)))
     )
@@
       (effects (font (size 1 1) (thickness 0.15)))
     )
-    (fp_text value 50k (at 0 1.55) (layer F.Fab)
-      (effects (font (size 1 1) (thickness 0.15)))
-    )
+    (fp_text value 18k (at 0 1.55) (layer F.Fab)
+      (effects (font (size 1 1) (thickness 0.15)))
+    )

Commit message: Continue iterating on layout.
Parts:
- C27, C28, C29, C31, C45, C46, R10, R14, R18, R21, R23, R26, R28, R30, R9, U5: moved to B.Cu
- moved C27 49.4 mm to (191.2, 84.6)
- moved C28 49.4 mm to (187.7, 84.6)
- moved R14 48.7 mm to (191.2, 85.7)
- moved C29 48.6 mm to (187.7, 85.9)
- moved R28 47.7 mm to (184.4, 88.0)
- moved C46 47.3 mm to (184.4, 89.2)
- moved R26 47.0 mm to (184.4, 90.5)
- moved C31 46.9 mm to (192.2, 91.2), turned to 90 degrees
- moved C45 46.9 mm to (194.8, 91.2), turned to 90 degrees
- moved R23 46.9 mm to (193.5, 91.2), turned to 270 degrees
- moved R30 46.9 mm to (188.9, 92.4)
- moved R25 20.6 mm to (153.0, 76.9), turned to 90 degrees
- moved C21 12.8 mm to (150.9, 101.5)
- moved TP6 12.7 mm to (137.2, 99.1)
- moved TP7 12.7 mm to (149.9, 99.1)
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Routing:
- net Net-(L3-Pad1): track 33.9 -> 0.00 mm, vias 3 -> 0
- net VOUT-: track 16.7 -> 43.1 mm
- net VOUT+: track 16.5 -> 41.5 mm
- net Net-(L4-Pad2): track 23.7 -> 7.34 mm
- net GNDA: track 101.9 -> 88.0 mm, vias 33 -> 30
- net /Analog/+1.65V: track 11.7 -> 0.00 mm, vias 2 -> 0
- net TRIGGER: track 43.5 -> 53.9 mm, vias 2 -> 4
- net Net-(C46-Pad1): track 5.31 -> 0.00 mm
- net +3V3: track 48.3 -> 43.7 mm, vias 24 -> 21
- net AMP0_EN: track 39.0 -> 42.7 mm
- net Net-(C31-Pad2): track 4.89 -> 1.74 mm
- net Net-(C27-Pad1): track 4.42 -> 1.80 mm
- net AMP1_EN: track 37.1 -> 39.5 mm
- net Net-(R19-Pad2): track 14.9 -> 12.7 mm
- net Net-(C32-Pad2): track 9.87 -> 8.00 mm
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